File: metuorbit.kicad_sch (KiCad schematic)
At the start: 29 parts, among them IC1 BLACKPILLF4, IC2 LoRa E220-900T30D, IC3 BNO055, IC4 NEO-M8N, IC5 BMP388, IC6 MicroSD_Reader, IC7 HT7333, IC8 MP1584, J1 Resistive Wire, J2 BATT Input, J3 SERVO1, J4 SERVO2, Q1 2N3904, Q2 IRLZ44N

Commit message: Traces and connecters are adjusted for ESC.
Parts:
- removed J4: SERVO2, Connector_PinHeader_2.54mm:PinHeader_1x03_P2.54mm_Vertical, symbol Connector:Conn_01x03_Pin
- added J4: ESC, symbol Connector:Conn_01x08_Pin
Connections:
- net LORA_AUX: now reaches IC2.5 (AUX)
- net LORA_AUX: now also IC1.PB8
- net SERVO2: no longer names the net of IC1.PB1
Other:
- note added: "UNFINISHED"
